Commit message: feat: contact/bumper sensor — ground-truth collision detection
Add a physics contact sensor to both robot templates, giving true
collision detection independent of the LiDAR-proximity heuristic. This
is a composable primitive: a new sensor, a new metric, a new assertion,
and a new episode event — the agent decides how to use them.

Integration (the fiddly part, now solved):
- URDF: a <sensor type=contact> on the base body, referencing the
  post-lumping collision name base_footprint_fixed_joint_lump__
  base_link_collision (verified via gz sdf -p).
- world: the gz-sim-contact-system plugin at world scope (it does not
  populate sensors from model scope).
- launch: the contact sensor ignores its SDF <topic> and publishes on
  the scoped gz path /world/warehouse/model/<robot>/link/base_footprint/
  sensor/bumper/contact; bridge that and ROS-remap it to /bumper.

Product wiring:
- metrics: contact_count (distinct contact episodes) from /bumper, in
  the whole-episode collector (ros_gz_interfaces/Contacts).
- assertion: no_contact (ground truth), alongside no_collision.
- episode events: use /bumper as the authoritative collision signal,
  falling back to the /scan heuristic when absent; episode query gets a
  Contacts formatter (num_contacts).
- stop-before-obstacle now asserts no_contact; manifests list the
  contact sensor; SCENARIO-FORMAT + ROADMAP + AGENTS updated.
- 2 new unit tests (39 total).

Verified E2E on BOTH templates: head-on collision publishes real
contacts on /bumper (690 msgs); stop-before-obstacle reports
contact_count=1 with no_contact failing; episode events shows the
ground-truth collision timestamp. On camera-bot, /image (98 frames) and
/bumper (3775 msgs) both record correctly. No image rebuild needed
(ros_gz_interfaces ships with the bridge).

Co-Authored-By: Claude Opus 4.8 <noreply@anthropic.com>

File: robotbase/templates/camera-bot/src/warehouse_bot_description/urdf/warehouse_bot.urdf.xacro (robot description, xacro)
@@ -132,3 +132,18 @@
     </sensor>
   </gazebo>
+  <!-- Contact/bumper sensor: ground-truth collision detection. Physics-based (no
+       rendering), so it runs headless like the rest. It references only the base body
+       collision — the box body is held off the floor by the wheels, so the sensor fires
+       when the robot hits something, not on the ground. The collision name is what
+       sdformat produces after lumping the base_link fixed joint into base_footprint.
+       The Contact *system* that feeds this sensor is declared at world scope (warehouse.sdf). -->
+  <gazebo reference="base_footprint">
+    <sensor name="bumper" type="contact">
+      <always_on>true</always_on>
+      <update_rate>30</update_rate>
+      <contact>
+        <collision>base_footprint_fixed_joint_lump__base_link_collision</collision>
+      </contact>
+    </sensor>
+  </gazebo>
 </robot>

File: robotbase/templates/differential-drive/src/warehouse_bot_description/urdf/warehouse_bot.urdf.xacro (robot description, xacro)
@@ -112,3 +112,18 @@
     </sensor>
   </gazebo>
+  <!-- Contact/bumper sensor: ground-truth collision detection. Physics-based (no
+       rendering), so it runs headless like the rest. It references only the base body
+       collision — the box body is held off the floor by the wheels, so the sensor fires
+       when the robot hits something, not on the ground. The collision name is what
+       sdformat produces after lumping the base_link fixed joint into base_footprint.
+       The Contact *system* that feeds this sensor is declared at world scope (warehouse.sdf). -->
+  <gazebo reference="base_footprint">
+    <sensor name="bumper" type="contact">
+      <always_on>true</always_on>
+      <update_rate>30</update_rate>
+      <contact>
+        <collision>base_footprint_fixed_joint_lump__base_link_collision</collision>
+      </contact>
+    </sensor>
+  </gazebo>
 </robot>

Commit message: feat: IMU sensor on the mobile templates (widening — sensors)
Add an IMU (orientation, angular velocity, linear acceleration) to
differential-drive and camera-bot: a world-scope gz Imu system + an
imu_link contact... sensor on the base, bridged to /imu
(sensor_msgs/Imu). Physics-based, headless. Exposed in the manifest and
via robotbase describe.

Verified E2E: /imu publishes at 50 Hz with a valid orientation quaternion
(robot upright -> identity).

Co-Authored-By: Claude Opus 4.8 <noreply@anthropic.com>

File: robotbase/templates/camera-bot/src/warehouse_bot_description/urdf/warehouse_bot.urdf.xacro (robot description, xacro)
@@ -75,4 +75,10 @@
     <origin xyz="${body_x/2 - 0.03} 0 ${body_z/2 + 0.03}"/>
   </joint>
+  <link name="imu_link"/>
+  <joint name="imu_joint" type="fixed">
+    <parent link="base_link"/>
+    <child link="imu_link"/>
+    <origin xyz="0 0 ${body_z/2}"/>
+  </joint>
   <link name="camera_link"/>
   <joint name="camera_joint" type="fixed">
@@ -118,4 +124,13 @@
     </sensor>
   </gazebo>
+  <!-- IMU: orientation, angular velocity, linear acceleration (physics-based). -->
+  <gazebo reference="imu_link">
+    <sensor name="imu" type="imu">
+      <topic>imu</topic>
+      <gz_frame_id>imu_link</gz_frame_id>
+      <update_rate>50</update_rate>
+      <always_on>true</always_on>
+    </sensor>
+  </gazebo>
   <gazebo reference="camera_link">
     <sensor name="camera" type="camera">

File: robotbase/templates/differential-drive/src/warehouse_bot_description/urdf/warehouse_bot.urdf.xacro (robot description, xacro)
@@ -75,5 +75,11 @@
     <origin xyz="${body_x/2 - 0.03} 0 ${body_z/2 + 0.03}"/>
   </joint>
-  <!-- Gazebo Harmonic: differential drive + friction + LiDAR -->
+  <link name="imu_link"/>
+  <joint name="imu_joint" type="fixed">
+    <parent link="base_link"/>
+    <child link="imu_link"/>
+    <origin xyz="0 0 ${body_z/2}"/>
+  </joint>
+  <!-- Gazebo Harmonic: differential drive + friction + LiDAR + IMU -->
   <gazebo>
     <plugin filename="gz-sim-diff-drive-system" name="gz::sim::systems::DiffDrive">
@@ -112,4 +118,14 @@
     </sensor>
   </gazebo>
+  <!-- IMU: orientation, angular velocity, linear acceleration. Physics-based (no
+       rendering); driven by the Imu system declared at world scope. -->
+  <gazebo reference="imu_link">
+    <sensor name="imu" type="imu">
+      <topic>imu</topic>
+      <gz_frame_id>imu_link</gz_frame_id>
+      <update_rate>50</update_rate>
+      <always_on>true</always_on>
+    </sensor>
+  </gazebo>
   <!-- Contact/bumper sensor: ground-truth collision detection. Physics-based (no
        rendering), so it runs headless like the rest. It references only the base body
