Commit message: refactor(ir): migrate emitters + compile onto the semantic IR (Tasks 7-9)
The modules (differential-drive/arm/quadrotor) and sensors now emit typed
RigidBody/Joint into the Fragment; compile_robot merges them into a RobotModel
(merge.build_model) and renders through backends.urdf.render_urdf. The string
renderer (merge.merge_and_render) is deleted; fixed_joint is now a Joint factory;
the raw-part escape hatch carries verbatim link XML via RigidBody.raw_xml (an
explicit, documented portability-breaking hatch — not used by the archetypes).

This is one atomic commit because Fragment cannot be half-typed: all producers had
to flip together for compile to build a RobotModel uniformly.

Golden regenerated once (per the 2026-07-31 decision): 7 URDF files change in
formatting only — compact links become verbose, and hand-authored literals
normalize through the one numeric formatter (0.10->0.1, 1e-5->1e-05, 0.0->0).
Proven behavior-preserving: under XML canonicalization + number normalization,
old vs new golden have ZERO semantic diffs (all SDFs and joints unchanged; the
custom-import ref is byte-identical). URDF is whitespace-insensitive between
elements and the numbers are equal to Gazebo's parser, so the sim loads identically.

249 offline tests pass.

Co-Authored-By: Claude Opus 4.8 <noreply@anthropic.com>

File: tests/golden/tpl-arm.urdf (robot description, URDF)
Before this commit: robot warehouse_bot, 5 links, 4 joints
Links:
- link arm_base_link: mass 10.0 -> 10; geometry collision cylinder length=0.1 radius=0.07; visual cylinder length=0.1 radius=0.07

File: tests/golden/tpl-drone.urdf (robot description, URDF)
Before this commit: robot warehouse_bot, 6 links, 5 joints
Links:
- link base_link: mass 1.0 -> 1
